Commit message: Update otter_gazebo.urdf.xacro

File: otter_gazebo/urdf/otter_gazebo.urdf.xacro (robot description, xacro)
@@ -10,4 +10,10 @@
   <xacro:arg name="ground_truth_enabled"  default="false" />
   <xacro:arg name="direct_control_plugin" default="false" />
+  <link name="dummy">
+   </link>
+  <joint name="dummy_joint" type="fixed">
+     <parent link="dummy"/>
+     <child link="base_link"/>
+   </joint>
   <!-- Define macros -->
   <!-- Defines the "otter_base" macro -->
